Commit message: first commit

File: turtlebot_arm_description/urdf/pincher_arm.urdf.xacro (robot description, xacro)
@@ -18,9 +18,43 @@
     <!-- As we don't have here a turtlebot base, add a base_link link as its location reference -->
     <link name="base_link"/>
+      <!-- Used for fixing robot to Gazebo 'base_link' -->
+  <link name="world"/>
+  <joint name="fixed" type="fixed">
+    <parent link="world"/>
+    <child link="base_link"/>
+  </joint>
+<!-- copy start: Copied from https://github.com/corot/thorp/blob/master/thorp_description/urdf/thorp_gazebo.urdf.xacro -->
+   <!-- Gazebo configuration for arm and cannon servos control -->
+  <gazebo>
+    <plugin name="gazebo_ros_control" filename="libgazebo_ros_control.so">
+      <!-- namespace added because of the inmoov example (https://github.com/MatthewVerbryke/inmoov_ros) -->
+      <robotNamespace>/turtlebot_arm</robotNamespace>
+      <!-- from: https://groups.google.com/forum/#%21topic/moveit-users/zNRG50tHuuY -->
+       <robotSimType>gazebo_ros_control/DefaultRobotHWSim</robotSimType>
+    </plugin>
+  </gazebo>
+  <xacro:macro name="servo_transmission" params="name">
+    <transmission name="${name}_trans">
+      <type>transmission_interface/SimpleTransmission</type>
+      <joint name="${name}_joint">
+        <hardwareInterface>hardware_interface/PositionJointInterface</hardwareInterface>
+      </joint>
+      <actuator name="${name}_motor">
+        <hardwareInterface>hardware_interface/PositionJointInterface</hardwareInterface>
+        <mechanicalReduction>1</mechanicalReduction>
+      </actuator>
+    </transmission>
+  </xacro:macro>
+  <servo_transmission name="arm_shoulder_pan"/>
+  <servo_transmission name="arm_shoulder_lift"/>
+  <servo_transmission name="arm_elbow_flex"/>
+  <servo_transmission name="arm_wrist_flex"/>
+  <servo_transmission name="gripper"/>
+  <!-- copy end -->
     <!-- Turtlebot arm macro -->
     <turtlebot_arm parent="base_link" color="Gray" gripper_color="Gray"   pincher_gripper="true" turtlebot_gripper="false">
       <!-- Place the "floating" arm at the location it should be if mounted on a turtlebot,
            as pick and place and other demos assume this location -->
-      <origin xyz="0.1 0.03 0.435"/>
+      <origin xyz="0 0 0.058"/> <!-- height of the PhantomX Pincher base = ca. 58mm -->
     </turtlebot_arm>
 </robot>

File: turtlebot_arm_description/urdf/turtlebot_arm.urdf.xacro (robot description, xacro)
@@ -17,4 +17,61 @@
     <!-- As we don't have here a turtlebot base, add a base_link link as its location reference -->
     <link name="base_link"/>
+    <!-- Used for fixing robot to Gazebo 'base_link' -->
+  <link name="world"/>
+  <joint name="fixed" type="fixed">
+    <parent link="world"/>
+    <child link="base_link"/>
+  </joint>
+<!-- copy start: Copied from https://github.com/corot/thorp/blob/master/thorp_description/urdf/thorp_gazebo.urdf.xacro -->
+   <!-- Gazebo configuration for arm and cannon servos control -->
+  <gazebo>
+    <plugin name="gazebo_ros_control" filename="libgazebo_ros_control.so">
+      <!-- namespace added because of the inmoov example (https://github.com/MatthewVerbryke/inmoov_ros) -->
+      <robotNamespace>/turtlebot_arm</robotNamespace>
+      <!-- from: https://groups.google.com/forum/#%21topic/moveit-users/zNRG50tHuuY -->
+       <robotSimType>gazebo_ros_control/DefaultRobotHWSim</robotSimType>
+    </plugin>
+  </gazebo>
+  <xacro:macro name="servo_transmission" params="name">
+    <transmission name="${name}_trans">
+      <type>transmission_interface/SimpleTransmission</type>
+      <joint name="${name}_joint">
+        <hardwareInterface>hardware_interface/PositionJointInterface</hardwareInterface>
+      </joint>
+      <actuator name="${name}_motor">
+        <hardwareInterface>hardware_interface/PositionJointInterface</hardwareInterface>
+        <mechanicalReduction>1</mechanicalReduction>
+      </actuator>
+    </transmission>
+  </xacro:macro>
+  <servo_transmission name="arm_shoulder_pan"/>
+  <servo_transmission name="arm_shoulder_lift"/>
+  <servo_transmission name="arm_elbow_flex"/>
+  <servo_transmission name="arm_wrist_flex"/>
+  <servo_transmission name="gripper"/>
+  <!-- <servo_transmission name="cannon"/> -->
+  <!-- Gazebo configuration for other structural parts -->
+  <xacro:macro name="structural_part" params="name color">
+    <gazebo reference="${name}_link">
+      <material>Gazebo/${color}</material>
+      <selfCollide>true</selfCollide>
+      <gravity>true</gravity>
+    </gazebo>
+  </xacro:macro>
+  <!-- <structural_part name="sonars_mount" color="Black"/>
+  <structural_part name="senz3d_mount" color="Black"/>
+  <structural_part name="xtion_mount"  color="Black"/>
+  <structural_part name="arm_mount"    color="Black"/>
+  <structural_part name="opencm"       color="Black"/>
+  <structural_part name="cannon"       color="Black"/>
+  <structural_part name="cannon_servo" color="Black"/>
+  <structural_part name="cannon_shaft" color="Black"/>
+  <structural_part name="cannon_tube1" color="Black"/>
+  <structural_part name="cannon_tube2" color="Black"/>
+  <structural_part name="cannon_tube3" color="Black"/>
+  <structural_part name="cannon_tube4" color="Black"/>
+  <structural_part name="cannon_tube5" color="Black"/>
+  <structural_part name="cannon_tube6" color="Black"/> -->
+  <!-- copy end -->
     <!-- Turtlebot arm macro -->
     <turtlebot_arm parent="base_link" color="White" gripper_color="Green"
